File: board/plc14500/SPRAM.sch (KiCad schematic (older format))
At the start: 31 parts, among them U14 4011, U15 4051

Commit message: Schematic tweaks
Parts:
- C15: renamed from C?; Price (none) -> 0.02
- C16, C17: Price (none) -> 0.02
- D43: renamed from D49; value LED5MM -> LED 5MM Red; Price (none) -> 0.01
- D44: renamed from D50; value LED5MM -> LED 5MM Red; Price (none) -> 0.01
- D45: renamed from D51; value LED5MM -> LED 5MM Red; Price (none) -> 0.01
- D46: renamed from D52; value LED5MM -> LED 5MM Red; Price (none) -> 0.01
- D47: renamed from D53; value LED5MM -> LED 5MM Red; Price (none) -> 0.01
- D48: renamed from D54; value LED5MM -> LED 5MM Red; Price (none) -> 0.01
- D49: renamed from D55; value LED5MM -> LED 5MM Red; Price (none) -> 0.01
- D50: renamed from D56; value LED5MM -> LED 5MM Red; Price (none) -> 0.01
- R59: renamed from R?; Price (none) -> 0.01
- R60: renamed from R65; Price (none) -> 0.01
- R61: renamed from R66; Price (none) -> 0.01
- R62: renamed from R67; Price (none) -> 0.01
- R63: renamed from R68; Price (none) -> 0.01
- R64: renamed from R69; Price (none) -> 0.01
- R65: renamed from R70; Price (none) -> 0.01
- R66: renamed from R71; Price (none) -> 0.01
- R67: renamed from R72; Price (none) -> 0.01
- U11, U3: renamed from U?; value 4011 -> 74HC14; footprint (none) -> Package_DIP:DIP-14_W7.62mm_LongPads; Price (none) -> 0.16
- U12: renamed from U?; footprint (none) -> Package_DIP:DIP-14_W7.62mm_LongPads; Price (none) -> 0.2
- U13: renamed from U14; value 4011 -> 4099; footprint (none) -> Package_DIP:DIP-16_W7.62mm_LongPads; Price (none) -> 0.57
- U3: renamed from U?; Price (none) -> 0.16
- renumbered U15 to U14
Connections:
- net D7: now also U11.1, U3.11; no longer U11.13, U3.9
- net W: now also U3.13; no longer U3.11
- net at U12.6: now also U3.10; no longer U3.8
- net at U12.12, U12.9: now also U3.12; no longer U3.10
- net at U12.13: now also U11.2; no longer U11.12
Other:
- note added: "0"
- note added: "1"
- note added: "D7"
- note added: "IN-WINH"
- note added: "OUT-WD"
- note added: "Read Inputs"
- note added: "Read Scratchpad RAM"
- note added: "SRAM-WD"
- note added: "SRAM-WINH"
- note added: "Scratchpad RAM"
- note added: "W"
- note added: "Write Inputs"
- note added: "Write Line Glue Logic"
- note added: "Write Scratchpad RAM"

Commit message: All components on the board! WIP
Parts:
- D43, D44, D45, D46, D47, D48, D49, D50: footprint plc14500:LED_5MM -> plc14500:LED_3MM
- R59, R60, R61, R62, R63, R64, R65, R66, R67: footprint Resistor_THT:R_Axial_DIN0309_L9.0mm_D3.2mm_P12.70mm_Horizontal -> Resistor_THT:R_Axial_DIN0204_L3.6mm_D1.6mm_P7.62mm_Horizontal
Changed lines of the file:
@@
 F 0 "D43" H 7500 3475 45  0000 L CNN
 F 1 "LED 5MM Red" H 7578 3611 45  0001 L CNN
-F 2 "plc14500:LED_5MM" V 7300 3650 20  0001 C CNN
+F 2 "plc14500:LED_3MM" V 7300 3650 20  0001 C CNN
 F 3 "" H 7500 3650 50  0001 C CNN
 F 4 "XXX-00000" H 7578 3516 60  0001 L CNN "Field4"
@@
 F 0 "D44" H 7675 3475 45  0000 L CNN
 F 1 "LED 5MM Red" H 7753 3611 45  0001 L CNN
-F 2 "plc14500:LED_5MM" V 7475 3650 20  0001 C CNN
+F 2 "plc14500:LED_3MM" V 7475 3650 20  0001 C CNN
 F 3 "" H 7675 3650 50  0001 C CNN
 F 4 "XXX-00000" H 7753 3516 60  0001 L CNN "Field4"
@@
 F 0 "D45" H 7850 3475 45  0000 L CNN
 F 1 "LED 5MM Red" H 7928 3611 45  0001 L CNN
-F 2 "plc14500:LED_5MM" V 7650 3650 20  0001 C CNN
+F 2 "plc14500:LED_3MM" V 7650 3650 20  0001 C CNN
 F 3 "" H 7850 3650 50  0001 C CNN
 F 4 "XXX-00000" H 7928 3516 60  0001 L CNN "Field4"
@@
 F 0 "D46" H 8025 3475 45  0000 L CNN
 F 1 "LED 5MM Red" H 8103 3611 45  0001 L CNN
-F 2 "plc14500:LED_5MM" V 7825 3650 20  0001 C CNN
+F 2 "plc14500:LED_3MM" V 7825 3650 20  0001 C CNN
 F 3 "" H 8025 3650 50  0001 C CNN
 F 4 "XXX-00000" H 8103 3516 60  0001 L CNN "Field4"
@@
 F 0 "D47" H 8200 3475 45  0000 L CNN
 F 1 "LED 5MM Red" H 8278 3611 45  0001 L CNN
-F 2 "plc14500:LED_5MM" V 8000 3650 20  0001 C CNN
+F 2 "plc14500:LED_3MM" V 8000 3650 20  0001 C CNN
 F 3 "" H 8200 3650 50  0001 C CNN
 F 4 "XXX-00000" H 8278 3516 60  0001 L CNN "Field4"
@@
 F 0 "D48" H 8375 3475 45  0000 L CNN
 F 1 "LED 5MM Red" H 8453 3611 45  0001 L CNN
-F 2 "plc14500:LED_5MM" V 8175 3650 20  0001 C CNN
+F 2 "plc14500:LED_3MM" V 8175 3650 20  0001 C CNN
 F 3 "" H 8375 3650 50  0001 C CNN
 F 4 "XXX-00000" H 8453 3516 60  0001 L CNN "Field4"
@@
 F 0 "D49" H 8550 3475 45  0000 L CNN
 F 1 "LED 5MM Red" H 8628 3611 45  0001 L CNN
-F 2 "plc14500:LED_5MM" V 8350 3650 20  0001 C CNN
+F 2 "plc14500:LED_3MM" V 8350 3650 20  0001 C CNN
 F 3 "" H 8550 3650 50  0001 C CNN
 F 4 "XXX-00000" H 8628 3516 60  0001 L CNN "Field4"
@@
 F 0 "R60" H 7475 3950 50  0000 R CNN
 F 1 "680R" V 7400 4200 50  0000 R CNN
-F 2 "Resistor_THT:R_Axial_DIN0309_L9.0mm_D3.2mm_P12.70mm_Horizontal" V 7430 4100 50  0001 C CNN
+F 2 "Resistor_THT:R_Axial_DIN0204_L3.6mm_D1.6mm_P7.62mm_Horizontal" V 7430 4100 50  0001 C CNN
 F 3 "~" H 7500 4100 50  0001 C CNN
 F 4 "0.01" H 7500 4100 50  0001 C CNN "Price"
@@
 F 0 "R61" H 7650 3950 50  0000 R CNN
 F 1 "680R" V 7575 4200 50  0000 R CNN
-F 2 "Resistor_THT:R_Axial_DIN0309_L9.0mm_D3.2mm_P12.70mm_Horizontal" V 7605 4100 50  0001 C CNN
+F 2 "Resistor_THT:R_Axial_DIN0204_L3.6mm_D1.6mm_P7.62mm_Horizontal" V 7605 4100 50  0001 C CNN
 F 3 "~" H 7675 4100 50  0001 C CNN
 F 4 "0.01" H 7675 4100 50  0001 C CNN "Price"
@@
 F 0 "R62" H 7825 3950 50  0000 R CNN
 F 1 "680R" V 7750 4200 50  0000 R CNN
-F 2 "Resistor_THT:R_Axial_DIN0309_L9.0mm_D3.2mm_P12.70mm_Horizontal" V 7780 4100 50  0001 C CNN
+F 2 "Resistor_THT:R_Axial_DIN0204_L3.6mm_D1.6mm_P7.62mm_Horizontal" V 7780 4100 50  0001 C CNN
 F 3 "~" H 7850 4100 50  0001 C CNN
 F 4 "0.01" H 7850 4100 50  0001 C CNN "Price"
@@
 F 0 "R63" H 8000 3950 50  0000 R CNN
 F 1 "680R" V 7925 4200 50  0000 R CNN
-F 2 "Resistor_THT:R_Axial_DIN0309_L9.0mm_D3.2mm_P12.70mm_Horizontal" V 7955 4100 50  0001 C CNN
+F 2 "Resistor_THT:R_Axial_DIN0204_L3.6mm_D1.6mm_P7.62mm_Horizontal" V 7955 4100 50  0001 C CNN
 F 3 "~" H 8025 4100 50  0001 C CNN
 F 4 "0.01" H 8025 4100 50  0001 C CNN "Price"
@@
 F 0 "R64" H 8175 3950 50  0000 R CNN
 F 1 "680R" V 8100 4200 50  0000 R CNN
-F 2 "Resistor_THT:R_Axial_DIN0309_L9.0mm_D3.2mm_P12.70mm_Horizontal" V 8130 4100 50  0001 C CNN
+F 2 "Resistor_THT:R_Axial_DIN0204_L3.6mm_D1.6mm_P7.62mm_Horizontal" V 8130 4100 50  0001 C CNN
 F 3 "~" H 8200 4100 50  0001 C CNN
 F 4 "0.01" H 8200 4100 50  0001 C CNN "Price"
@@
 F 0 "R65" H 8350 3950 50  0000 R CNN
 F 1 "680R" V 8275 4200 50  0000 R CNN
-F 2 "Resistor_THT:R_Axial_DIN0309_L9.0mm_D3.2mm_P12.70mm_Horizontal" V 8305 4100 50  0001 C CNN
+F 2 "Resistor_THT:R_Axial_DIN0204_L3.6mm_D1.6mm_P7.62mm_Horizontal" V 8305 4100 50  0001 C CNN
 F 3 "~" H 8375 4100 50  0001 C CNN
 F 4 "0.01" H 8375 4100 50  0001 C CNN "Price"
@@
 F 0 "R66" H 8525 3950 50  0000 R CNN
 F 1 "680R" V 8450 4200 50  0000 R CNN
-F 2 "Resistor_THT:R_Axial_DIN0309_L9.0mm_D3.2mm_P12.70mm_Horizontal" V 8480 4100 50  0001 C CNN
+F 2 "Resistor_THT:R_Axial_DIN0204_L3.6mm_D1.6mm_P7.62mm_Horizontal" V 8480 4100 50  0001 C CNN
 F 3 "~" H 8550 4100 50  0001 C CNN
 F 4 "0.01" H 8550 4100 50  0001 C CNN "Price"
@@
 F 0 "D50" H 8725 3475 45  0000 L CNN
 F 1 "LED 5MM Red" H 8803 3611 45  0001 L CNN
-F 2 "plc14500:LED_5MM" V 8525 3650 20  0001 C CNN
+F 2 "plc14500:LED_3MM" V 8525 3650 20  0001 C CNN
 F 3 "" H 8725 3650 50  0001 C CNN
 F 4 "XXX-00000" H 8803 3516 60  0001 L CNN "Field4"
@@
 F 0 "R67" H 8700 3950 50  0000 R CNN
 F 1 "680R" V 8625 4200 50  0000 R CNN
-F 2 "Resistor_THT:R_Axial_DIN0309_L9.0mm_D3.2mm_P12.70mm_Horizontal" V 8655 4100 50  0001 C CNN
+F 2 "Resistor_THT:R_Axial_DIN0204_L3.6mm_D1.6mm_P7.62mm_Horizontal" V 8655 4100 50  0001 C CNN
 F 3 "~" H 8725 4100 50  0001 C CNN
 F 4 "0.01" H 8725 4100 50  0001 C CNN "Price"
@@
 F 0 "R59" H 1450 3225 50  0000 R CNN
 F 1 "680R" V 1375 3475 50  0000 R CNN
-F 2 "Resistor_THT:R_Axial_DIN0309_L9.0mm_D3.2mm_P12.70mm_Horizontal" V 1405 3375 50  0001 C CNN
+F 2 "Resistor_THT:R_Axial_DIN0204_L3.6mm_D1.6mm_P7.62mm_Horizontal" V 1405 3375 50  0001 C CNN
 F 3 "~" H 1475 3375 50  0001 C CNN
 F 4 "0.01" H 1475 3375 50  0001 C CNN "Price"
@@
 F 4 "0.16" H 1850 3100 50  0001 C CNN "Price"
 	3    1850 3100
-	1    0    0    -1
-$EndComp
-$Comp
-L 74xx:74HC14 U?
-U 4 1 67AF2AEC
-P 2450 3100
-AR Path="/67AF2AEC" Ref="U?"  Part="1"
-AR Path="/63B4BDA9/67AF2AEC" Ref="U?"  Part="4"
-AR Path="/67425B3B/67AF2AEC" Ref="U11"  Part="4"
-F 0 "U11" H 2550 2975 50  0000 C CNN
-F 1 "74HC14" H 2625 2900 50  0000 C CNN
-F 2 "Package_DIP:DIP-14_W7.62mm_LongPads" H 2450 3100 50  0001 C CNN
-F 3 "http://www.intersil.com/content/dam/Intersil/documents/cd40/cd4011bms-12bms-23bms.pdf" H 2450 3100 50  0001 C CNN
-F 4 "0.16" H 2450 3100 50  0001 C CNN "Price"
-	4    2450 3100
 	1    0    0    -1
 $EndComp
@@
 Wire Notes Line
 	2675 6100 4650 6100
+$Comp
+L 74xx:74HC14 U?
+U 4 1 67AF2AEC
+P 2450 3100
+AR Path="/67AF2AEC" Ref="U?"  Part="1"
+AR Path="/63B4BDA9/67AF2AEC" Ref="U?"  Part="4"
+AR Path="/67425B3B/67AF2AEC" Ref="U11"  Part="4"
+F 0 "U11" H 2550 2975 50  0000 C CNN
+F 1 "74HC14" H 2625 2900 50  0000 C CNN
+F 2 "Package_DIP:DIP-14_W7.62mm_LongPads" H 2450 3100 50  0001 C CNN
+F 3 "http://www.intersil.com/content/dam/Intersil/documents/cd40/cd4011bms-12bms-23bms.pdf" H 2450 3100 50  0001 C CNN
+F 4 "0.16" H 2450 3100 50  0001 C CNN "Price"
+	4    2450 3100
+	1    0    0    -1
+$EndComp
 Wire Bus Line
 	9300 3700 9300 4100
