File: board/plc14500/plc14500.kicad_pcb (KiCad board)
At the start: 2 copper layers, 135 parts, among them U1 74HC14, U2 4051, U3 74HC14, U4 Arduino Nano, U5 CD4099, U6 NE555, U7 74HC590A, U8 LH5168, U9 MC14500

Commit message: Schematic tweaks
Parts:
- removed S19: SW_Push, Button_Switch_THT:SW_Tactile_Straight_KSA0Axx1LFTR
- removed S20: SWITCH-DPDT-PTH-GPI-152-3013, plc14500:SWITCH_DPDT
- added C12: 100nF, Capacitor_THT:C_Rect_L7.2mm_W2.5mm_P5.00mm_FKS2_FKP2_MKS2_MKP2, F.Cu at (381.1, 128.2)
- added C13: 100nF, Capacitor_THT:C_Rect_L7.2mm_W2.5mm_P5.00mm_FKS2_FKP2_MKS2_MKP2, F.Cu at (376.9, 124.2)
- added C14: 100nF, Capacitor_THT:C_Rect_L7.2mm_W2.5mm_P5.00mm_FKS2_FKP2_MKS2_MKP2, F.Cu at (326.8, 162.2)
- added C15: 100nF, Capacitor_THT:C_Rect_L7.2mm_W2.5mm_P5.00mm_FKS2_FKP2_MKS2_MKP2, F.Cu at (484.4, 44.3)
- added C16: 100nF, Capacitor_THT:C_Rect_L7.2mm_W2.5mm_P5.00mm_FKS2_FKP2_MKS2_MKP2, F.Cu at (477.0, 54.2)
- added C17: 100nF, Capacitor_THT:C_Rect_L7.2mm_W2.5mm_P5.00mm_FKS2_FKP2_MKS2_MKP2, F.Cu at (469.7, 58.9)
- added D41: LED 5MM Red, plc14500:LED_5MM, F.Cu at (385.0, 159.2)
- added D42: LED 5MM Red, plc14500:LED_5MM, F.Cu at (493.7, 46.0)
- added D43: LED 5MM Red, plc14500:LED_5MM, F.Cu at (494.0, 61.1)
- added D44: LED 5MM Red, plc14500:LED_5MM, F.Cu at (486.5, 61.1)
- added D45: LED 5MM Red, plc14500:LED_5MM, F.Cu at (494.0, 53.6)
- added D46: LED 5MM Red, plc14500:LED_5MM, F.Cu at (470.3, 64.7)
- added D47: LED 5MM Red, plc14500:LED_5MM, F.Cu at (479.0, 60.0)
- added D48: LED 5MM Red, plc14500:LED_5MM, F.Cu at (477.8, 67.5)
- added D49: LED 5MM Red, plc14500:LED_5MM, F.Cu at (486.5, 53.6)
- added R56: 680R, Resistor_THT:R_Axial_DIN0309_L9.0mm_D3.2mm_P12.70mm_Horizontal, F.Cu at (376.6, 119.8)
- added R57: 680R, Resistor_THT:R_Axial_DIN0309_L9.0mm_D3.2mm_P12.70mm_Horizontal, F.Cu at (484.1, 35.1)
- added R58: 680R, Resistor_THT:R_Axial_DIN0309_L9.0mm_D3.2mm_P12.70mm_Horizontal, F.Cu at (484.1, 39.9)
- added R59: 680R, Resistor_THT:R_Axial_DIN0309_L9.0mm_D3.2mm_P12.70mm_Horizontal, F.Cu at (453.5, 68.8)
- added R60: 680R, Resistor_THT:R_Axial_DIN0309_L9.0mm_D3.2mm_P12.70mm_Horizontal, F.Cu at (453.5, 64.0)
- added R61: 680R, Resistor_THT:R_Axial_DIN0309_L9.0mm_D3.2mm_P12.70mm_Horizontal, F.Cu at (437.7, 66.5)
- added R62: 680R, Resistor_THT:R_Axial_DIN0309_L9.0mm_D3.2mm_P12.70mm_Horizontal, F.Cu at (453.5, 59.3)
- added R63: 680R, Resistor_THT:R_Axial_DIN0309_L9.0mm_D3.2mm_P12.70mm_Horizontal, F.Cu at (460.9, 54.5)
- added R64: 680R, Resistor_THT:R_Axial_DIN0309_L9.0mm_D3.2mm_P12.70mm_Horizontal, F.Cu at (437.7, 61.8)
- added R65: 680R, Resistor_THT:R_Axial_DIN0309_L9.0mm_D3.2mm_P12.70mm_Horizontal, F.Cu at (437.7, 57.0)
- added RV1: 10K, Potentiometer_THT:Potentiometer_ACP_CA9-H5_Horizontal, F.Cu at (353.6, 91.1)
- added U10: MC14500, Package_DIP:DIP-16_W7.62mm_LongPads, F.Cu at (333.7, 105.2)
- added U11: 74HC14, Package_DIP:DIP-14_W7.62mm_LongPads, F.Cu at (461.3, 34.8)
- added U12: 4011, Package_DIP:DIP-14_W7.62mm_LongPads, F.Cu at (472.9, 34.8)
- added U13: 4099, Package_DIP:DIP-16_W7.62mm_LongPads, F.Cu at (438.1, 34.8)
- added U14: 4051, Package_DIP:DIP-16_W7.62mm_LongPads, F.Cu at (449.7, 34.8)
- C4: value C -> 10uF; footprint Capacitor_THT:C_Rect_L7.2mm_W2.5mm_P5.00mm_FKS2_FKP2_MKS2_MKP2 -> Capacitor_THT:CP_Radial_D8.0mm_P5.00mm
- C5, C8: value C -> 100nF
- C7: value 100nF -> 10uF; footprint Capacitor_THT:C_Rect_L7.2mm_W2.5mm_P5.00mm_FKS2_FKP2_MKS2_MKP2 -> Capacitor_THT:CP_Radial_D8.0mm_P5.00mm
- D1, D10, D11, D12, D13, D14, D15, D16, D17, D18, D19, D2, D20, D21, D22, D23, D24, D25, D26, D27, D28, D29, D3, D30, D31, D32, D33, D34, D35, D36, D37, D38, D39, D4, D40, D5, D6, D7, D8, D9: value LED5MM -> LED 5MM Red
- R12, R21: value 47K -> 680R
- R25: value 680R -> 47K
- R42, R46: value 10K -> 680R
- R48, R49: value 680R -> 10K
- R52: value 680R -> 1K
- S1, S10, S11, S17, S2, S3, S4, S9: value SW_Push -> Push Button
- S12: value SW_Push -> Switch DPDT; footprint Button_Switch_THT:SW_Tactile_Straight_KSA0Axx1LFTR -> plc14500:SWITCH_DPDT
- S13, S14, S16, S18, S5, S6, S7, S8: value SWITCH-DPDT-PTH-GPI-152-3013 -> Switch DPDT
- S15: value SWITCH-DPDT-PTH-GPI-152-3013 -> Push Button; footprint plc14500:SWITCH_DPDT -> Button_Switch_THT:SW_Tactile_Straight_KSA0Axx1LFTR
- U4: value Arduino Nano -> NE555; footprint Module:Arduino_Nano -> Package_DIP:DIP-8_W7.62mm
- U5: value CD4099 -> 4099
- U6: value NE555 -> Arduino Nano; footprint Package_DIP:DIP-8_W7.62mm -> Module:Arduino_Nano
- U9: value MC14500 -> NE555; footprint Package_DIP:DIP-16_W7.62mm_LongPads -> Package_DIP:DIP-8_W7.62mm
- moved C4 319.0 mm to (404.0, 59.0)
- moved R48 311.5 mm to (392.4, 110.3)
- moved C6 300.4 mm to (425.8, 38.8)
- moved U9 298.9 mm to (372.1, 133.7)
- moved U1 288.5 mm to (357.8, 34.8)
- moved R13 288.2 mm to (369.0, 39.9)
- moved C5 286.3 mm to (392.6, 70.5)
- moved C9 285.7 mm to (408.6, 109.2)
- moved D26 281.2 mm to (406.3, 131.5)
- moved D11 280.7 mm to (421.3, 62.0)
- moved R25 280.6 mm to (369.0, 35.1)
- moved C1 279.1 mm to (425.8, 34.8)
- moved U4 273.8 mm to (342.4, 90.0)
- moved R4 273.6 mm to (365.9, 64.0)
- moved D15 272.5 mm to (413.8, 62.0)
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Connections:
- net Net-(D10-PadA) renamed OUT6
- net Net-(D11-PadA) renamed OUT5
- net Net-(D12-PadA) renamed OUT4
- net Net-(D13-PadA) renamed OUT3
- C10 pad 1: GND -> Net-(C10-Pad1)
- C10 pad 2: Net-(C10-Pad2) -> GND
- C11 pad 1: +5V -> Net-(C11-Pad1)
- C2 pad 1: Net-(C2-Pad1) -> GND
- C2 pad 2: W -> +5V
- C3 pad 1: +5V -> GND
- C3 pad 2: GND -> +5V
- C4 pad 1: Net-(C4-Pad1) -> (no net)
- C4 pad 2: GND -> (no net)
- C5 pad 1: Net-(C5-Pad1) -> +5V
- C7 pad 1: GND -> (no net)
- C7 pad 2: +5V -> (no net)
- C8 pad 1: Net-(C8-Pad1) -> +5V
- D14 pad A: RES -> OUT2
- D15 pad A: Net-(D15-PadA) -> OUT1
- D16 pad A: Net-(D16-PadA) -> OUT0
- D17 pad A: Net-(D17-PadA) -> RES
- D20 pad A: Net-(D20-PadA) -> A0
- D21 pad A: A0 -> D0
- D22 pad A: D0 -> A1
- D23 pad A: A1 -> D1
- D24 pad A: D1 -> A2
- D25 pad A: Net-(D25-PadA) -> D2
- D26 pad A: A2 -> A3
- D27 pad A: D2 -> D3
- D28 pad A: A3 -> Net-(D28-PadA)
- D29 pad A: D3 -> A4
- D30 pad A: A4 -> D4
- D31 pad A: D4 -> A5
- D32 pad A: A5 -> D5
- D33 pad A: D5 -> Net-(D33-PadA)
- D37 pad A: Net-(D37-PadA) -> CLK
- D40 pad A: W -> Net-(D40-PadA)
- D8 pad A: /Input/Output/IN7 -> IN7
- D9 pad A: Net-(D9-PadA) -> TMR0-TRG
- R12 pad 2: Net-(R12-Pad2) -> Net-(D5-PadK)
- R13 pad 2: Net-(D5-PadK) -> Net-(D6-PadK)
- R14 pad 2: Net-(D6-PadK) -> Net-(D7-PadK)
- R15 pad 1: GND -> Net-(R15-Pad1)
- R15 pad 2: Net-(D7-PadK) -> Net-(C4-Pad+)
- R16 pad 1: GND -> Net-(D8-PadK)
- R16 pad 2: Net-(D8-PadK) -> GND
- R17 pad 2: Net-(C2-Pad1) -> Net-(D9-PadK)
- R18 pad 2: Net-(D9-PadK) -> Net-(D10-PadK)
- R19 pad 2: Net-(D10-PadK) -> Net-(D11-PadK)
- R20 pad 2: Net-(D11-PadK) -> Net-(D12-PadK)
- R21 pad 1: +5V -> GND
- R21 pad 2: Net-(D14-PadK) -> Net-(D13-PadK)
- R22 pad 2: Net-(D12-PadK) -> Net-(D14-PadK)
- R23 pad 2: Net-(D13-PadK) -> Net-(D15-PadK)
- R24 pad 2: Net-(D15-PadK) -> Net-(D16-PadK)
- R25 pad 1: +5V -> RES
- R25 pad 2: RES -> GND
- R26 pad 1: GND -> Net-(D17-PadK)
- R26 pad 2: Net-(D16-PadK) -> GND
- R27 pad 1: GND -> Net-(R27-Pad1)
- R27 pad 2: Net-(D17-PadK) -> Net-(D19-PadA)
- R28 pad 2: Net-(D19-PadA) -> Net-(D18-PadA)
- R29 pad 2: Net-(D18-PadA) -> +5V
- R30 pad 1: Net-(R30-Pad1) -> Net-(R29-Pad1)
- R30 pad 2: +5V -> Net-(C10-Pad1)
- R31 pad 1: Net-(R30-Pad1) -> GND
- R31 pad 2: Net-(C5-Pad1) -> Net-(D20-PadK)
- R32 pad 2: Net-(D20-PadK) -> Net-(D21-PadK)
- R33 pad 2: Net-(D21-PadK) -> Net-(D22-PadK)
- R34 pad 2: Net-(D22-PadK) -> Net-(D23-PadK)
- R35 pad 2: Net-(D23-PadK) -> Net-(D24-PadK)
- R36 pad 2: Net-(D24-PadK) -> Net-(D25-PadK)
- R37 pad 2: Net-(D25-PadK) -> Net-(D26-PadK)
- R38 pad 2: Net-(D26-PadK) -> Net-(D27-PadK)
- R39 pad 2: Net-(D27-PadK) -> Net-(D28-PadK)
- R40 pad 2: Net-(D28-PadK) -> Net-(D29-PadK)
- R41 pad 2: Net-(D29-PadK) -> Net-(D30-PadK)
- R42 pad 1: Net-(R42-Pad1) -> GND
- R42 pad 2: +5V -> Net-(D31-PadK)
- R43 pad 2: Net-(D30-PadK) -> Net-(D32-PadK)
- R44 pad 2: Net-(D31-PadK) -> Net-(D33-PadK)
- R45 pad 2: Net-(D32-PadK) -> Net-(D34-PadK)
- R46 pad 1: Net-(C10-Pad2) -> GND
- R46 pad 2: Net-(R42-Pad1) -> Net-(D35-PadK)
- R47 pad 2: Net-(D33-PadK) -> Net-(D36-PadK)
- R48 pad 1: GND -> Net-(R48-Pad1)
- R48 pad 2: Net-(D34-PadK) -> +5V
- R49 pad 1: GND -> Net-(C13-Pad2)
- R49 pad 2: Net-(D35-PadK) -> Net-(R48-Pad1)
- R50 pad 2: Net-(D36-PadK) -> Net-(D37-PadK)
- R52 pad 1: GND -> RES
- R52 pad 2: Net-(D37-PadK) -> Net-(D38-PadA)
- S12 pad 1: Net-(R12-Pad2) -> Net-(S12-Pad1)
- S12 pad 2: +5V -> /Input/Output/IN4
- S13 pad 1: (no net) -> Net-(S13-Pad1)
- S13 pad 2: (no net) -> /Input/Output/IN5
- S13 pad 3: (no net) -> Net-(S13-Pad3)
- S13 pad 6: Net-(R9-Pad2) -> Net-(R10-Pad2)
- S13 pad 7: /Input/Output/IN4 -> Net-(S13-Pad3)
- S14 pad 1: (no net) -> Net-(S14-Pad1)
- S14 pad 2: (no net) -> /Input/Output/IN6
- S14 pad 3: (no net) -> Net-(S14-Pad3)
- S14 pad 6: Net-(R10-Pad2) -> Net-(R11-Pad2)
- S14 pad 7: /Input/Output/IN5 -> Net-(S14-Pad3)
- S15 pad 1: (no net) -> RES
- S15 pad 2: (no net) -> +5V
- S16 pad 1: (no net) -> Net-(R27-Pad1)
- S16 pad 2: (no net) -> +5V
- S16 pad 3: (no net) -> Net-(R28-Pad1)
- S16 pad 5: Net-(S16-Pad5) -> Net-(C10-Pad1)
- S16 pad 6: Net-(R12-Pad2) -> (no net)
- S16 pad 7: /Input/Output/IN7 -> (no net)
- S17 pad 2: Net-(D14-PadK) -> Net-(R48-Pad1)
- S18 pad 1: Net-(R28-Pad1) -> Net-(S18-Pad1)
- S18 pad 2: +5V -> CLK
- S18 pad 3: Net-(R29-Pad1) -> Net-(S18-Pad3)
- S18 pad 5: Net-(C5-Pad1) -> Net-(D33-PadA)
- S18 pad 6: Net-(C4-Pad1) -> +5V
- S18 pad 7: (no net) -> Net-(D28-PadA)
- S5 pad 1: (no net) -> Net-(S5-Pad1)
- S5 pad 2: (no net) -> /Input/Output/IN0
- S5 pad 3: (no net) -> Net-(S5-Pad3)
- S5 pad 7: /Input/Output/IN0 -> Net-(S5-Pad3)
- S6 pad 1: (no net) -> Net-(S6-Pad1)
- S6 pad 2: (no net) -> /Input/Output/IN1
- S6 pad 3: (no net) -> Net-(S6-Pad3)
- S6 pad 7: /Input/Output/IN1 -> Net-(S6-Pad3)
- S7 pad 1: (no net) -> Net-(S7-Pad1)
- S7 pad 2: (no net) -> /Input/Output/IN2
- S7 pad 3: (no net) -> Net-(S7-Pad3)
- S7 pad 7: /Input/Output/IN2 -> Net-(S7-Pad3)
- S8 pad 1: (no net) -> Net-(S8-Pad1)
- S8 pad 2: (no net) -> /Input/Output/IN3
- S8 pad 3: (no net) -> Net-(S8-Pad3)
- S8 pad 7: /Input/Output/IN3 -> Net-(S8-Pad3)
- U1 pad 10: /Input/Output/IN4 -> Net-(S12-Pad1)
- U1 pad 11: Net-(S13-Pad5) -> Net-(S12-Pad5)
- U1 pad 12: /Input/Output/IN5 -> Net-(S13-Pad1)
- U1 pad 13: Net-(S14-Pad5) -> Net-(S13-Pad5)
- U1 pad 2: /Input/Output/IN0 -> Net-(S5-Pad1)
- U1 pad 4: /Input/Output/IN1 -> Net-(S6-Pad1)
- U1 pad 6: /Input/Output/IN2 -> Net-(S7-Pad1)
- U1 pad 8: /Input/Output/IN3 -> Net-(S8-Pad1)
- U2 pad 4: /Input/Output/IN7 -> IN7
- U2 pad 6: W -> IN-WINH
- U3 pad 1: Net-(S15-Pad5) -> Net-(S14-Pad5)
- U3 pad 10: (no net) -> Net-(U12-Pad6)
- U3 pad 11: (no net) -> D7
- U3 pad 12: (no net) -> Net-(U12-Pad12)
- U3 pad 13: (no net) -> W
- U3 pad 2: /Input/Output/IN6 -> Net-(S14-Pad1)
- U3 pad 3: Net-(S16-Pad5) -> RES
- U3 pad 4: /Input/Output/IN7 -> !RES
- U3 pad 5: Net-(C2-Pad1) -> Net-(C15-Pad1)
- U3 pad 6: Net-(U3-Pad6) -> Net-(U11-Pad9)
- U3 pad 8: Net-(S20-Pad1) -> Net-(S18-Pad1)
- U3 pad 9: Net-(C10-Pad2) -> Net-(C13-Pad2)
- U4 pad 1: (no net) -> GND
- U4 pad 2: (no net) -> TMR0-TRG
- U4 pad 3: Net-(D14-PadK) -> IN7
- U4 pad 4: GND -> !RES
- U4 pad 5: D0 -> (no net)
- U4 pad 6: D1 -> Net-(C4-Pad+)
- U4 pad 7: D2 -> Net-(C4-Pad+)
- U4 pad 8: D3 -> +5V
- U5 pad 1: Net-(D9-PadA) -> TMR0-TRG
- U5 pad 10: Net-(D16-PadA) -> OUT1
- U5 pad 11: Net-(D15-PadA) -> OUT2
- U5 pad 4: Net-(U3-Pad6) -> OUT-WD
- U5 pad 9: Net-(D17-PadA) -> OUT0
- U6 pad 1: GND -> (no net)
- U6 pad 2: Net-(C5-Pad1) -> (no net)
- U6 pad 3: Net-(S20-Pad3) -> (no net)
- U6 pad 4: +5V -> GND
- U6 pad 5: Net-(C8-Pad1) -> D0
- U6 pad 6: Net-(C5-Pad1) -> D1
- U6 pad 7: Net-(R30-Pad1) -> D2
- U6 pad 8: +5V -> D3
- U9 pad 1: CLK -> GND
- U9 pad 2: W -> Net-(C10-Pad1)
- U9 pad 3: D -> Net-(S18-Pad3)
- U9 pad 4: D3 -> +5V
- U9 pad 5: D2 -> Net-(C11-Pad1)
- U9 pad 6: D1 -> Net-(C10-Pad1)
- U9 pad 7: D0 -> Net-(R29-Pad1)
- U9 pad 8: GND -> +5V
Other:
- board outline added: 160.1 x 100.1 mm

Commit message: All components on the board! WIP
Parts:
- added C18: 100nF, Capacitor_THT:C_Rect_L7.2mm_W2.5mm_P5.00mm_FKS2_FKP2_MKS2_MKP2, F.Cu at (77.6, 100.8)
- added C19: 100nF, Capacitor_THT:C_Rect_L7.2mm_W2.5mm_P5.00mm_FKS2_FKP2_MKS2_MKP2, F.Cu at (102.7, 100.8)
- added D50: LED 5MM Red, plc14500:LED_3MM, F.Cu at (204.1, 86.2)
- added R66: 680R, Resistor_THT:R_Axial_DIN0204_L3.6mm_D1.6mm_P7.62mm_Horizontal, F.Cu at (200.2, 75.4)
- added R67: 680R, Resistor_THT:R_Axial_DIN0204_L3.6mm_D1.6mm_P7.62mm_Horizontal, F.Cu at (205.3, 75.4)
- D1, D10, D11, D12, D13, D14, D15, D16, D17, D18, D19, D2, D20, D21, D22, D23, D24, D25, D26, D27, D28, D29, D3, D30, D31, D32, D33, D34, D35, D36, D37, D38, D39, D4, D40, D41, D42, D43, D44, D45, D46, D47, D48, D49, D5, D6, D7, D8, D9: footprint plc14500:LED_5MM -> plc14500:LED_3MM
- R1, R10, R11, R12, R13, R14, R15, R16, R17, R18, R19, R2, R20, R21, R23, R24, R27, R28, R29, R3, R30, R31, R32, R33, R34, R35, R36, R37, R38, R39, R4, R40, R41, R42, R43, R44, R45, R46, R47, R5, R55, R56, R57, R58, R59, R6, R60, R61, R62, R63, R64, R65, R7, R8, R9: footprint Resistor_THT:R_Axial_DIN0309_L9.0mm_D3.2mm_P12.70mm_Horizontal -> Resistor_THT:R_Axial_DIN0204_L3.6mm_D1.6mm_P7.62mm_Horizontal
- R22: value 680R -> 0R; footprint Resistor_THT:R_Axial_DIN0309_L9.0mm_D3.2mm_P12.70mm_Horizontal -> Resistor_THT:R_Axial_DIN0204_L3.6mm_D1.6mm_P7.62mm_Horizontal
- R25: value 47K -> 680R; footprint Resistor_THT:R_Axial_DIN0309_L9.0mm_D3.2mm_P12.70mm_Horizontal -> Resistor_THT:R_Axial_DIN0204_L3.6mm_D1.6mm_P7.62mm_Horizontal
- R26: value 680R -> 47K; footprint Resistor_THT:R_Axial_DIN0309_L9.0mm_D3.2mm_P12.70mm_Horizontal -> Resistor_THT:R_Axial_DIN0204_L3.6mm_D1.6mm_P7.62mm_Horizontal
- R48, R49: value 10K -> 680R; footprint Resistor_THT:R_Axial_DIN0309_L9.0mm_D3.2mm_P12.70mm_Horizontal -> Resistor_THT:R_Axial_DIN0204_L3.6mm_D1.6mm_P7.62mm_Horizontal
- R50: value 680R -> 10K; footprint Resistor_THT:R_Axial_DIN0309_L9.0mm_D3.2mm_P12.70mm_Horizontal -> Resistor_THT:R_Axial_DIN0204_L3.6mm_D1.6mm_P7.62mm_Horizontal
- R51: value 1M -> 10K; footprint Resistor_THT:R_Axial_DIN0309_L9.0mm_D3.2mm_P12.70mm_Horizontal -> Resistor_THT:R_Axial_DIN0204_L3.6mm_D1.6mm_P7.62mm_Horizontal
- R52: value 1K -> 680R; footprint Resistor_THT:R_Axial_DIN0309_L9.0mm_D3.2mm_P12.70mm_Horizontal -> Resistor_THT:R_Axial_DIN0204_L3.6mm_D1.6mm_P7.62mm_Horizontal
- R53: value 680R -> 1M; footprint Resistor_THT:R_Axial_DIN0309_L9.0mm_D3.2mm_P12.70mm_Horizontal -> Resistor_THT:R_Axial_DIN0204_L3.6mm_D1.6mm_P7.62mm_Horizontal
- R54: value 680R -> 1K; footprint Resistor_THT:R_Axial_DIN0309_L9.0mm_D3.2mm_P12.70mm_Horizontal -> Resistor_THT:R_Axial_DIN0204_L3.6mm_D1.6mm_P7.62mm_Horizontal
- U6: moved to B.Cu
- moved C15 391.3 mm to (100.0, 117.5)
- moved U11 384.5 mm to (82.7, 102.1), turned to 90 degrees
- moved U12 372.2 mm to (106.8, 102.1), turned to 90 degrees
- moved C1 356.9 mm to (77.6, 113.0), turned to 90 degrees
- moved C16 351.6 mm to (127.9, 95.8), turned to 270 degrees
- moved R59 344.0 mm to (113.0, 117.5)
- moved D42 341.6 mm to (154.5, 86.2)
- moved D1 336.6 mm to (84.9, 122.3)
- moved R57 335.9 mm to (150.6, 75.4), turned to 270 degrees
- moved D2 335.9 mm to (99.6, 122.3)
- moved C9 331.8 mm to (77.6, 85.0), turned to 90 degrees
- moved S2 331.3 mm to (97.1, 128.5)
- moved R58 330.3 mm to (155.7, 75.4), turned to 270 degrees
- moved D43 326.6 mm to (168.4, 86.2)
- moved S6 322.5 mm to (96.9, 141.1), turned to 90 degrees
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Connections:
- net OUT0 renamed Net-(D16-PadA)
- net OUT1 renamed Net-(D15-PadA)
- net OUT2 renamed Net-(D14-PadA)
- net OUT3 renamed Net-(D13-PadA)
- net OUT4 renamed Net-(D12-PadA)
- net OUT5 renamed Net-(D11-PadA)
- net OUT6 renamed Net-(D10-PadA)
- C4 pad 1: (no net) -> Net-(C4-Pad1)
- C4 pad 2: (no net) -> GND
- C7 pad 1: (no net) -> Net-(C7-Pad1)
- C7 pad 2: (no net) -> GND
- D37 pad A: CLK -> D7
- D38 pad A: Net-(D38-PadA) -> CLK
- D41 pad A: W -> Net-(D41-PadA)
- D42 pad A: Net-(D42-PadA) -> W
- R15 pad 2: Net-(C4-Pad+) -> Net-(C4-Pad1)
- R22 pad 1: GND -> +5V
- R22 pad 2: Net-(D14-PadK) -> Net-(R22-Pad2)
- R23 pad 2: Net-(D15-PadK) -> Net-(D14-PadK)
- R24 pad 2: Net-(D16-PadK) -> Net-(D15-PadK)
- R25 pad 1: RES -> GND
- R25 pad 2: GND -> Net-(D16-PadK)
- R26 pad 1: Net-(D17-PadK) -> RES
- R27 pad 1: Net-(R27-Pad1) -> Net-(D17-PadK)
- R27 pad 2: Net-(D19-PadA) -> GND
- R28 pad 2: Net-(D18-PadA) -> Net-(D19-PadA)
- R29 pad 2: +5V -> Net-(D18-PadA)
- R30 pad 1: Net-(R29-Pad1) -> Net-(R30-Pad1)
- R30 pad 2: Net-(C10-Pad1) -> +5V
- R31 pad 1: GND -> Net-(R30-Pad1)
- R31 pad 2: Net-(D20-PadK) -> Net-(C10-Pad1)
- R32 pad 2: Net-(D21-PadK) -> Net-(D20-PadK)
- R33 pad 2: Net-(D22-PadK) -> Net-(D21-PadK)
- R34 pad 2: Net-(D23-PadK) -> Net-(D22-PadK)
- R35 pad 2: Net-(D24-PadK) -> Net-(D23-PadK)
- R36 pad 2: Net-(D25-PadK) -> Net-(D24-PadK)
- R37 pad 2: Net-(D26-PadK) -> Net-(D25-PadK)
- R38 pad 2: Net-(D27-PadK) -> Net-(D26-PadK)
- R39 pad 2: Net-(D28-PadK) -> Net-(D27-PadK)
- R40 pad 2: Net-(D29-PadK) -> Net-(D28-PadK)
- R41 pad 2: Net-(D30-PadK) -> Net-(D29-PadK)
- R42 pad 2: Net-(D31-PadK) -> Net-(D30-PadK)
- R43 pad 2: Net-(D32-PadK) -> Net-(D31-PadK)
- R44 pad 2: Net-(D33-PadK) -> Net-(D32-PadK)
- R45 pad 2: Net-(D34-PadK) -> Net-(D33-PadK)
- R46 pad 2: Net-(D35-PadK) -> Net-(D34-PadK)
- R47 pad 2: Net-(D36-PadK) -> Net-(D35-PadK)
- R48 pad 1: Net-(R48-Pad1) -> GND
- R48 pad 2: +5V -> Net-(D36-PadK)
- R49 pad 1: Net-(C13-Pad2) -> GND
- R49 pad 2: Net-(R48-Pad1) -> Net-(D37-PadK)
- R50 pad 1: GND -> Net-(R50-Pad1)
- R50 pad 2: Net-(D37-PadK) -> +5V
- R51 pad 1: Net-(R51-Pad1) -> Net-(C13-Pad2)
- R51 pad 2: CLK -> Net-(R50-Pad1)
- R52 pad 1: RES -> GND
- R52 pad 2: Net-(D38-PadA) -> Net-(D38-PadK)
- R53 pad 1: GND -> Net-(R53-Pad1)
- R53 pad 2: Net-(D38-PadK) -> CLK
- R54 pad 1: GND -> RES
- R54 pad 2: Net-(D39-PadK) -> Net-(D39-PadA)
- R55 pad 2: Net-(D40-PadK) -> Net-(D39-PadK)
- R56 pad 2: Net-(D41-PadK) -> Net-(D40-PadK)
- R57 pad 2: Net-(C15-Pad1) -> Net-(D41-PadK)
- R59 pad 2: Net-(D43-PadK) -> Net-(C15-Pad1)
- R60 pad 2: Net-(D44-PadK) -> Net-(D43-PadK)
- R61 pad 2: Net-(D45-PadK) -> Net-(D44-PadK)
- R62 pad 2: Net-(D46-PadK) -> Net-(D45-PadK)
- R63 pad 2: Net-(D47-PadK) -> Net-(D46-PadK)
- R64 pad 2: Net-(D48-PadK) -> Net-(D47-PadK)
- R65 pad 2: Net-(D49-PadK) -> Net-(D48-PadK)
- S16 pad 1: Net-(R27-Pad1) -> Net-(R28-Pad1)
- S16 pad 3: Net-(R28-Pad1) -> Net-(R29-Pad1)
- S16 pad 6: (no net) -> Net-(C7-Pad1)
- S17 pad 2: Net-(R48-Pad1) -> Net-(R50-Pad1)
- U1 pad 14: (no net) -> +5V
- U1 pad 7: (no net) -> GND
- U10 pad 10: Net-(D39-PadA) -> Net-(D40-PadA)
- U10 pad 14: Net-(R51-Pad1) -> Net-(R53-Pad1)
- U10 pad 15: Net-(D40-PadA) -> Net-(D41-PadA)
- U10 pad 9: Net-(D38-PadA) -> Net-(D39-PadA)
- U11 pad 14: (no net) -> +5V
- U11 pad 7: (no net) -> GND
- U12 pad 14: (no net) -> +5V
- U12 pad 7: (no net) -> GND
- U13 pad 1: Net-(D49-PadA) -> Net-(D50-PadA)
- U13 pad 10: Net-(D43-PadA) -> Net-(D44-PadA)
- U13 pad 11: Net-(D44-PadA) -> Net-(D45-PadA)
- U13 pad 12: Net-(D45-PadA) -> Net-(D46-PadA)
- U13 pad 13: Net-(D46-PadA) -> Net-(D47-PadA)
- U13 pad 14: Net-(D47-PadA) -> Net-(D48-PadA)
- U13 pad 15: Net-(D48-PadA) -> Net-(D49-PadA)
- U13 pad 5: /SPRAM/D4 -> D4
- U13 pad 6: /SPRAM/D5 -> D5
- U13 pad 7: /SPRAM/D6 -> D6
- U13 pad 9: Net-(D42-PadA) -> Net-(D43-PadA)
- U14 pad 1: Net-(D46-PadA) -> Net-(D47-PadA)
- U14 pad 10: /SPRAM/D5 -> D5
- U14 pad 11: /SPRAM/D4 -> D4
- U14 pad 12: Net-(D45-PadA) -> Net-(D46-PadA)
- U14 pad 13: Net-(D42-PadA) -> Net-(D43-PadA)
- U14 pad 14: Net-(D43-PadA) -> Net-(D44-PadA)
- U14 pad 15: Net-(D44-PadA) -> Net-(D45-PadA)
- U14 pad 2: Net-(D48-PadA) -> Net-(D49-PadA)
- U14 pad 4: Net-(D49-PadA) -> Net-(D50-PadA)
- U14 pad 5: Net-(D47-PadA) -> Net-(D48-PadA)
- U14 pad 9: /SPRAM/D6 -> D6
- U3 pad 14: (no net) -> +5V
- U3 pad 7: (no net) -> GND
- U4 pad 6: Net-(C4-Pad+) -> Net-(C4-Pad1)
- U4 pad 7: Net-(C4-Pad+) -> Net-(C4-Pad1)
- U6 pad 27: +5V -> Net-(R22-Pad2)
- U8 pad 19: (no net) -> D7
- U9 pad 7: Net-(R29-Pad1) -> Net-(R30-Pad1)
Routing:
- net (no net): vias 0 -> 5
Other:
- board size 160.1 x 100.1 mm -> 160.1 x 99.9 mm
- board text added: "0"
- board text added: "7"
- board text added: "ADDR"
- board text added: "CLK"
- board text added: "DATA"
- board text added: "F"
- board text added: "HI"
- board text added: "IN0"
- board text added: "IN1"
- board text added: "IN2"
- board text added: "IN3"
- board text added: "IN4"
- board text added: "IN5"
- board text added: "IN6"
- board text added: "IN7"
- board text added: "LO"
- board text added: "O"
- board text added: "OUT0"
- board text added: "OUT1"
- board text added: "OUT2"
- board text added: "OUT3"
- board text added: "OUT4"
- board text added: "OUT5"
- board text added: "OUT6"
- board text added: "OUT7"
- board text added: "R"
- board text added: "RR"
- board text added: "RST"
- board text added: "RUN"
- board text added: "SPR"
- board text added: "ST"
- board text added: "STEP"
- board text added: "TMR0"
- board text added: "W"
