File: board/plc14500/plc14500.kicad_pcb (KiCad board)
At the start: 2 copper layers, 160.1 x 101 mm, 174 parts, among them U1 74HC14, U10 MC14500, U11 74HC14, U12 4011, U13 4099, U14 4051, U2 4051, U3 74HC14, U4 NE555, U5 4099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

Commit message: Cleanup REV.D
Parts:
- D33: value LED 3MM Red -> LED 3MM Yellow
- D41, D52: value LED 3MM Red -> LED 3MM Orange
Changed lines of the file:
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@@
         (effects (font (size 1 1) (thickness 0.15)))
     )
+    (fp_text user "${VALUE}" (at -20.955 33.02) (layer "F.Fab")
+        (effects (font (size 1 1) (thickness 0.15)))
+    )
+    (fp_text user "${VALUE}" (at -20.955 17.78) (layer "F.Fab")
+        (effects (font (size 1 1) (thickness 0.15)))
+    )
     (fp_line (start -0.29 -1.236) (end -0.29 -1.08)
       (stroke (width 0.12) (type solid)) (layer "F.SilkS"))
@@
         (effects (font (size 1 1) (thickness 0.15)))
     )
-    (fp_text value "LED 3MM Red" (at -9.93 -3.3) (layer "F.Fab")
+    (fp_text value "LED 3MM Yellow" (at -4.44 -3.3) (layer "F.Fab")
         (effects (font (size 1 1) (thickness 0.15)))
     )
@@
         (effects (font (size 1 1) (thickness 0.15)))
     )
-    (fp_text value "LED 3MM Red" (at 1.27 2.96) (layer "F.Fab")
+    (fp_text value "LED 3MM Orange" (at 1.27 2.96) (layer "F.Fab")
         (effects (font (size 1 1) (thickness 0.15)))
     )
@@
         (effects (font (size 1 1) (thickness 0.15)))
     )
-    (fp_text value "LED 3MM Red" (at 1.27 2.96) (layer "F.Fab")
-        (effects (font (size 1 1) (thickness 0.15)))
-    )
-    (fp_text user "${VALUE}" (at 29.165 3.175) (layer "F.Fab")
-        (effects (font (size 1 1) (thickness 0.15)))
-    )
-    (fp_text user "${VALUE}" (at 27.895 -12.065) (layer "F.Fab")
+    (fp_text value "LED 3MM Orange" (at 1.27 2.96) (layer "F.Fab")
         (effects (font (size 1 1) (thickness 0.15)))
     )
