File: board/plc14500/plc14500.kicad_pcb (KiCad board)
At the start: 2 copper layers, 160.1 x 101 mm, 174 parts, among them U1 74HC14, U10 MC14500, U11 74HC14, U12 4011, U13 4099, U14 4051, U2 4051, U3 74HC14, U4 NE555, U5 4099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

Commit message: Fix/rst line (#20)
* Clear OUT and SPR on program

* Fix RST line pulsing on program upload doesn't work

* Bump bootloader version to 1.3
Parts:
- removed C20: 1uF NP, Capacitor_THT:C_Radial_D6.3mm_H5.0mm_P2.50mm
- D18, D19, D28, D38: value LED 3MM Red -> LED 3MM Yellow
- D39, D42, D50, D53: value LED 3MM Red -> LED 3MM Orange
Routing:
- net /PRG: track 130.9 -> 106.0 mm, vias 2 -> 0
- net /RES: track 268.2 -> 249.6 mm
Changed lines of the file:
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@@
         (effects (font (size 1 1) (thickness 0.15)))
     )
-    (fp_text value "LED 3MM Red" (at 1.27 2.96) (layer "F.Fab") hide
+    (fp_text value "LED 3MM Yellow" (at 1.27 2.96) (layer "F.Fab") hide
         (effects (font (size 1 1) (thickness 0.15)))
     )
@@
         (effects (font (size 1 1) (thickness 0.15)))
     )
-    (fp_text value "LED 3MM Red" (at 1.27 2.96) (layer "F.Fab") hide
+    (fp_text value "LED 3MM Yellow" (at 1.27 2.96) (layer "F.Fab") hide
         (effects (font (size 1 1) (thickness 0.15)))
     )
@@
         (effects (font (size 1 1) (thickness 0.15)))
     )
-    (fp_text value "LED 3MM Red" (at 1.27 2.96) (layer "F.Fab") hide
+    (fp_text value "LED 3MM Yellow" (at 1.27 2.96) (layer "F.Fab") hide
         (effects (font (size 1 1) (thickness 0.15)))
     )
@@
         (effects (font (size 1 1) (thickness 0.15)))
     )
-    (fp_text value "LED 3MM Red" (at 1.27 2.96) (layer "F.Fab") hide
+    (fp_text value "LED 3MM Yellow" (at 1.27 2.96) (layer "F.Fab") hide
         (effects (font (size 1 1) (thickness 0.15)))
     )
@@
         (effects (font (size 1 1) (thickness 0.15)))
     )
-    (fp_text value "LED 3MM Red" (at 1.27 2.96) (layer "F.Fab") hide
+    (fp_text value "LED 3MM Orange" (at 1.27 2.96) (layer "F.Fab") hide
         (effects (font (size 1 1) (thickness 0.15)))
     )
@@
         (effects (font (size 1 1) (thickness 0.15)))
     )
-    (fp_text value "LED 3MM Red" (at 1.27 2.96) (layer "F.Fab") hide
+    (fp_text value "LED 3MM Orange" (at 1.27 2.96) (layer "F.Fab") hide
         (effects (font (size 1 1) (thickness 0.15)))
     )
@@
         (effects (font (size 1 1) (thickness 0.15)))
     )
-    (fp_text value "LED 3MM Red" (at 1.27 2.96) (layer "F.Fab") hide
+    (fp_text value "LED 3MM Orange" (at 1.27 2.96) (layer "F.Fab") hide
         (effects (font (size 1 1) (thickness 0.15)))
     )
@@
     )
   )
-  (footprint "Capacitor_THT:C_Radial_D6.3mm_H5.0mm_P2.50mm" (layer "F.Cu")
-    (at 115.61 52.705)
-    (descr "C, Radial series, Radial, pin pitch=2.50mm, diameter=6.3mm, height=5mm, Non-Polar Electrolytic Capacitor")
-    (tags "C Radial series Radial pin pitch 2.50mm diameter 6.3mm height 5mm Non-Polar Electrolytic Capacitor")
-    (property "Sheetfile" "programming_if.kicad_sch")
-    (property "Sheetname" "Programming Interface")
-    (property "ki_description" "Unpolarized capacitor, small symbol")
-    (property "ki_keywords" "capacitor cap")
-    (attr through_hole)
-    (fp_text reference "C20" (at 1.23 1.905) (layer "F.SilkS")
-        (effects (font (size 1 1) (thickness 0.15)))
-    )
-    (fp_text value "1uF NP" (at 1.25 1.27) (layer "F.Fab")
-        (effects (font (size 1 1) (thickness 0.15)))
-    )
-    (fp_circle (center 1.25 0) (end 4.52 0)
-      (stroke (width 0.12) (type solid)) (fill none) (layer "F.SilkS"))
-    (fp_circle (center 1.25 0) (end 4.65 0)
-      (stroke (width 0.05) (type solid)) (fill none) (layer "F.CrtYd"))
-    (fp_circle (center 1.25 0) (end 4.4 0)
-      (stroke (width 0.1) (type solid)) (fill none) (layer "F.Fab"))
-    (pad "1" thru_hole circle (at 0 0) (size 1.6 1.6) (drill 0.8) (layers "*.Cu" "*.Mask")
-      (net 136 "/PRG") (pintype "passive"))
-    (pad "2" thru_hole circle (at 2.5 0) (size 1.6 1.6) (drill 0.8) (layers "*.Cu" "*.Mask")
-      (net 37 "/RES") (pintype "passive"))
-    (model "${KICAD6_3DMODEL_DIR}/Capacitor_THT.3dshapes/C_Radial_D6.3mm_H5.0mm_P2.50mm.wrl"
-      (offset (xyz 0 0 0))
-      (scale (xyz 1 1 1))
-      (rotate (xyz 0 0 0))
-    )
-  )
   (footprint "plc14500:LED_3MM" locked (layer "F.Cu")
     (at 154.395 86.36)
@@
         (effects (font (size 1 1) (thickness 0.15)))
     )
-    (fp_text value "LED 3MM Red" (at 1.27 2.96) (layer "F.Fab") hide
+    (fp_text value "LED 3MM Orange" (at 1.27 2.96) (layer "F.Fab") hide
         (effects (font (size 1 1) (thickness 0.15)))
     )
@@
   (segment (start 229.105 62.2152) (end 227.85 60.96) (width 0.25) (layer "B.Cu") (net 36))
   (segment (start 205.84 107.498) (end 205.84 108.262) (width 0.25) (layer "B.Cu") (net 36))
-  (segment (start 101.3508 48.7) (end 104.3911 51.7403) (width 0.25) (layer "F.Cu") (net 37))
   (segment (start 151.917 100.603) (end 150.122 100.603) (width 0.25) (layer "F.Cu") (net 37))
   (segment (start 194.41 115.101) (end 195.215 115.906) (width 0.25) (layer "F.Cu") (net 37))
   (segment (start 190.6 114.355) (end 190.6 112.828) (width 0.25) (layer "F.Cu") (net 37))
   (segment (start 223.08 111.024) (end 223.626 111.57) (width 0.25) (layer "F.Cu") (net 37))
-  (segment (start 114.126 51.5722) (end 116.9772 51.5722) (width 0.25) (layer "F.Cu") (net 37))
   (segment (start 137.151 99.3268) (end 139.016 101.192) (width 0.25) (layer "F.Cu") (net 37))
   (segment (start 149.448 101.277) (end 149.448 102.765) (width 0.25) (layer "F.Cu") (net 37))
@@
   (segment (start 195.215 115.906) (end 201.218 115.906) (width 0.25) (layer "F.Cu") (net 37))
   (segment (start 97.4231 55.5688) (end 97.4231 55.31) (width 0.25) (layer "F.Cu") (net 37))
-  (segment (start 104.3911 51.7403) (end 113.9579 51.7403) (width 0.25) (layer "F.Cu") (net 37))
-  (segment (start 113.9579 51.7403) (end 114.126 51.5722) (width 0.25) (layer "F.Cu") (net 37))
   (segment (start 190.6 112.828) (end 193.623 112.828) (width 0.25) (layer "F.Cu") (net 37))
   (segment (start 204.563 111.024) (end 223.08 111.024) (width 0.25) (layer "F.Cu") (net 37))
@@
   (segment (start 188.06 102.13) (end 188.06 103.657) (width 0.25) (layer "F.Cu") (net 37))
   (segment (start 154.97 103.657) (end 151.917 100.603) (width 0.25) (layer "F.Cu") (net 37))
-  (segment (start 116.9772 51.5722) (end 118.11 52.705) (width 0.25) (layer "F.Cu") (net 37))
   (segment (start 202.026 115.098) (end 202.026 113.561) (width 0.25) (layer "F.Cu") (net 37))
   (segment (start 223.626 113.559) (end 222.25 114.935) (width 0.25) (layer "F.Cu") (net 37))
@@
   (segment (start 97.93 74.91) (end 97.93 76.0369) (width 0.25) (layer "F.Cu") (net 136))
   (segment (start 163.683 91.1518) (end 165.514 92.9831) (width 0.25) (layer "F.Cu") (net 136))
-  (segment (start 97.5991 61.5031) (end 108.7665 61.5031) (width 0.25) (layer "F.Cu") (net 136))
   (segment (start 97.93 76.0369) (end 98.2117 76.0369) (width 0.25) (layer "F.Cu") (net 136))
   (segment (start 150.966 89.699) (end 152.582 88.0825) (width 0.25) (layer "F.Cu") (net 136))
   (segment (start 152.582 88.0825) (end 155.652 91.1518) (width 0.25) (layer "F.Cu") (net 136))
-  (segment (start 97.1551 61.9471) (end 97.5991 61.5031) (width 0.25) (layer "F.Cu") (net 136))
-  (segment (start 108.7665 61.5031) (end 108.7972 61.5338) (width 0.25) (layer "F.Cu") (net 136))
   (segment (start 112.796 91.398) (end 150.279 91.398) (width 0.25) (layer "F.Cu") (net 136))
-  (via (at 108.7972 61.5338) (size 0.8) (drill 0.4) (layers "F.Cu" "B.Cu") (net 136))
-  (via (at 97.1551 61.9471) (size 0.8) (drill 0.4) (layers "F.Cu" "B.Cu") (net 136))
-  (segment (start 97.28 63.2737) (end 97.1551 63.1488) (width 0.25) (layer "B.Cu") (net 136))
   (segment (start 97.28 73.1331) (end 97.93 73.7831) (width 0.25) (layer "B.Cu") (net 136))
   (segment (start 95.4571 54.1681) (end 96.47 54.1681) (width 0.25) (layer "B.Cu") (net 136))
   (segment (start 93.47 55.31) (end 94.5969 55.31) (width 0.25) (layer "B.Cu") (net 136))
   (segment (start 94.5969 55.31) (end 94.5969 55.0283) (width 0.25) (layer "B.Cu") (net 136))
-  (segment (start 97.1551 63.1488) (end 97.1551 61.9471) (width 0.25) (layer "B.Cu") (net 136))
   (segment (start 96.47 54.1681) (end 97.28 54.9781) (width 0.25) (layer "B.Cu") (net 136))
   (segment (start 94.5969 55.0283) (end 95.4571 54.1681) (width 0.25) (layer "B.Cu") (net 136))
-  (segment (start 115.61 54.721) (end 115.61 52.705) (width 0.25) (layer "B.Cu") (net 136))
-  (segment (start 108.7972 61.5338) (end 115.61 54.721) (width 0.25) (layer "B.Cu") (net 136))
   (segment (start 97.28 54.9781) (end 97.28 63.2737) (width 0.25) (layer "B.Cu") (net 136))
   (segment (start 97.28 63.2737) (end 97.28 73.1331) (width 0.25) (layer "B.Cu") (net 136))
