File: board/plc14500/CPU.sch (KiCad schematic (older format))
At the start: 73 parts, among them U10 MC14500, U11 74HC14, U3 74HC14, U7 74HC590A, U8 LH5168, U9 NE555

Commit message: rev.c board
Connections:
- net RR: now reaches D41.A, U10.15 (RR)
Changed lines of the file:
@@
 Sheet 3 4
 Title "PLC14500 - Nano"
-Date "2022-11-09"
-Rev "0.4"
+Date "2023-03-04"
+Rev "0.5"
 Comp "Nicola Cimmino"
-Comment1 ""
+Comment1 "REV.C"
 Comment2 ""
 Comment3 ""
@@
 Text Notes 750  3250 0    50   ~ 0
 Fhi = 1.44 / (R30+2×R31) × C10\nFhi = 4.8KHz\n\nFlo = 1.44 / (R30+2×R31) × (C10+C7)\nFlo = 1Hz
+Text GLabel 10550 3900 2    50   Output ~ 0
+RR
+Wire Wire Line
+	10275 3900 10550 3900
 Wire Bus Line
 	7800 3650 7800 4100
@@
 Wire Bus Line
 	3475 3800 3475 4975
+Connection ~ 10275 3900
 $EndSCHEMATC
