File: board/plc14500/CPU.kicad_sch (KiCad schematic)
At the start: 78 parts, among them U10 MC14500, U11 74HC14, U3 74HC14, U7 74HC590A, U8 LH5168, U9 NE555

Commit message: Cleanup REV.D
Parts:
- D18, D19, D28, D33, D38: value LED 3MM Red -> LED 3MM Yellow
- D39, D41, D42, D50, D52, D53: value LED 3MM Red -> LED 3MM Orange
Changed lines of the file:
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@@
       (effects (font (size 1.143 1.143)) (justify left))
     )
-    (property "Value" "LED 3MM Red" (at 126.4412 41.6306 0)
+    (property "Value" "LED 3MM Yellow" (at 126.4412 41.6306 0)
       (effects (font (size 1.143 1.143)) (justify left) hide)
     )
@@
       (effects (font (size 1.143 1.143)) (justify left))
     )
-    (property "Value" "LED 3MM Red" (at 134.0612 41.6306 0)
+    (property "Value" "LED 3MM Yellow" (at 134.0612 41.6306 0)
       (effects (font (size 1.143 1.143)) (justify left) hide)
     )
@@
       (effects (font (size 1.143 1.143)) (justify left))
     )
-    (property "Value" "LED 3MM Red" (at 57.8612 58.1406 0)
+    (property "Value" "LED 3MM Yellow" (at 57.8612 58.1406 0)
       (effects (font (size 1.143 1.143)) (justify left) hide)
     )
@@
       (effects (font (size 1.143 1.143)) (justify left))
     )
-    (property "Value" "LED 3MM Red" (at 62.9412 58.1406 0)
+    (property "Value" "LED 3MM Yellow" (at 62.9412 58.1406 0)
       (effects (font (size 1.143 1.143)) (justify left) hide)
     )
@@
       (effects (font (size 1.143 1.143)) (justify left))
     )
-    (property "Value" "LED 3MM Red" (at 192.4812 134.3406 0)
+    (property "Value" "LED 3MM Orange" (at 192.4812 134.3406 0)
       (effects (font (size 1.143 1.143)) (justify left) hide)
     )
@@
       (effects (font (size 1.143 1.143)) (justify left))
     )
-    (property "Value" "LED 3MM Red" (at 197.5612 134.3406 0)
+    (property "Value" "LED 3MM Orange" (at 197.5612 134.3406 0)
       (effects (font (size 1.143 1.143)) (justify left) hide)
     )
@@
       (effects (font (size 1.143 1.143)) (justify left))
     )
-    (property "Value" "LED 3MM Red" (at 202.6412 134.3406 0)
+    (property "Value" "LED 3MM Orange" (at 202.6412 134.3406 0)
       (effects (font (size 1.143 1.143)) (justify left) hide)
     )
@@
       (effects (font (size 1.143 1.143)) (justify left))
     )
-    (property "Value" "LED 3MM Red" (at 191.2112 53.0606 0)
+    (property "Value" "LED 3MM Yellow" (at 191.2112 53.0606 0)
       (effects (font (size 1.143 1.143)) (justify left) hide)
     )
@@
       (effects (font (size 1.143 1.143)) (justify left))
     )
-    (property "Value" "LED 3MM Red" (at 177.2412 134.3406 0)
+    (property "Value" "LED 3MM Orange" (at 177.2412 134.3406 0)
       (effects (font (size 1.143 1.143)) (justify left) hide)
     )
@@
       (effects (font (size 1.143 1.143)) (justify left))
     )
-    (property "Value" "LED 3MM Red" (at 187.4012 134.3406 0)
+    (property "Value" "LED 3MM Orange" (at 187.4012 134.3406 0)
       (effects (font (size 1.143 1.143)) (justify left) hide)
     )
@@
       (effects (font (size 1.143 1.143)) (justify left))
     )
-    (property "Value" "LED 3MM Red" (at 182.3212 134.3406 0)
+    (property "Value" "LED 3MM Orange" (at 182.3212 134.3406 0)
       (effects (font (size 1.143 1.143)) (justify left) hide)
     )
