File: board/plc14500/CPU.kicad_sch (KiCad schematic)
At the start: 73 parts, among them U10 MC14500, U11 74HC14, U3 74HC14, U7 74HC590A, U8 LH5168, U9 NE555

Commit message: Feature/rev.d (#19)
* First tests for a rust upload tool, WIP

* Rearrange LEDs

* Remove kicad backups

* REV.D Schema updates

* Restore PCB anchoring holes

* Address ERC errors

* Cleanup, ready to route

* REV.D first proto

* Fix issues on REV.D0

* REV.D schema fixes, better assembler output, some docs

* Add ignore of kicad lock files

* Fixes

* route

* Re-route REV.D, fab files next round

* Re-route REV.D, fab files next round

* Rev.d

* Added reset cap from program line

* REV.D artifacts

* Cleanup REV.D

* Remove old file
Parts:
- added D50, D52, D53: LED 3MM Orange, plc14500:LED_3MM, symbol plc14500:LED
- added R56, R67: 820R, Resistor_THT:R_Axial_DIN0204_L3.6mm_D1.6mm_P7.62mm_Horizontal, symbol Device:R
- C7: footprint Capacitor_THT:CP_Radial_D8.0mm_P5.00mm -> Capacitor_THT:CP_Radial_D5.0mm_P2.50mm; symbol plc14500-rescue:CP-Device -> plc14500:CP-Device
- D18, D19, D28, D33, D38: value LED 3MM Red -> LED 3MM Yellow; symbol plc14500-rescue:LED5MM-SparkFun-LED -> plc14500:LED; Field4 XXX-00000 -> (none)
- D20, D21, D22, D23, D24, D25, D26, D27, D29, D30, D31, D32, D34, D35, D36, D37: symbol plc14500-rescue:LED5MM-SparkFun-LED -> plc14500:LED; Field4 XXX-00000 -> (none)
- D39, D41, D42: value LED 3MM Red -> LED 3MM Orange; symbol plc14500-rescue:LED5MM-SparkFun-LED -> plc14500:LED; Field4 XXX-00000 -> (none)
- S16, S18: symbol plc14500-rescue:SWITCH-DPDT-PTH-GPI-152-3013-SparkFun-Switches -> plc14500:SWITCH-DPDT
- U11, U3: symbol 74xx:74HC14 -> plc14500:74HC14
- U7: symbol 74xx:74HC590A -> plc14500:74HC590A
- U8: symbol Memory_RAM:KM62256CLP -> plc14500:KM62256CLP
- U9: symbol plc14500-rescue:555D-SparkFun-IC-Special-Function -> plc14500:555
Connections:
- net GND: now also R53.1, S16.8 (GND), S16.9 (GND), S18.8 (GND), S18.9 (GND), R56.1, R67.1
- net at R30.1, U9.7 (DIS): now also R31.2; no longer R31.1
- net at C10.1, U9.2 (TRI), U9.6 (TRE): now also R31.1, S16.7; no longer R31.2, S16.5
- net at U9.3 (OUT): now also S18.1; no longer S18.3
- net at U3.8: now also S18.3; no longer S18.1
- net at S18.5: now also D28.A; no longer D33.A
- net at S18.7: now also D33.A; no longer D28.A
- net at S16.1: now also R29.1; no longer R28.1
- net at S16.3: now also R28.1; no longer R29.1
- net at U10.10 (FLAG0): now also D52.A
- net at U10.11 (RTN): now also D50.A
- net CLK1: now reaches U10.14 (X1)
- net CLK1: now also U7.11 (CPC), U7.13 (CPR); no longer R53.1
- net at U10.9 (FLAGF): now also D53.A
- net CLK renamed CLK2
- net CLK2: no longer R53.2, U7.11 (CPC), U7.13 (CPR)
- net WEN renamed !WEN
- new net: D50.K (C), R53.2
- new net: D53.K (C), R67.2
- new net: D52.K (C), R56.2
- no-connect marks 5 -> 2
Other:
- note added: "Program Memory"
- note removed: "Memory"
- moved on the sheet: C10, C11, C12, C13, C14, C7, C8, C9, D18, D19, D20, D21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
