File: board/plc14500/IO.kicad_sch (KiCad schematic)
At the start: 71 parts, among them U1 74HC14, U2 4051, U3 74HC14, U5 4099, U6 Arduino Nano

Commit message: Feature/rev.d (#19)
* First tests for a rust upload tool, WIP

* Rearrange LEDs

* Remove kicad backups

* REV.D Schema updates

* Restore PCB anchoring holes

* Address ERC errors

* Cleanup, ready to route

* REV.D first proto

* Fix issues on REV.D0

* REV.D schema fixes, better assembler output, some docs

* Add ignore of kicad lock files

* Fixes

* route

* Re-route REV.D, fab files next round

* Re-route REV.D, fab files next round

* Rev.d

* Added reset cap from program line

* REV.D artifacts

* Cleanup REV.D

* Remove old file
Parts:
- removed D17: LED 3MM Red, plc14500:LED_3MM, symbol plc14500-rescue:LED5MM-SparkFun-LED
- removed R26: 47K, Resistor_THT:R_Axial_DIN0204_L3.6mm_D1.6mm_P7.62mm_Horizontal, symbol Device:R
- removed R27: 820R, Resistor_THT:R_Axial_DIN0204_L3.6mm_D1.6mm_P7.62mm_Horizontal, symbol Device:R
- removed S15: Push Button, plc14500:SW_Tactile_THT, symbol Switch:SW_Push
- removed unit 2 of U3
- removed U6: Arduino Nano, Module:Arduino_Nano, symbol MCU_Module:Arduino_Nano_v2.x
- added C1, C2: 100nF, Capacitor_THT:C_Rect_L7.2mm_W2.5mm_P5.00mm_FKS2_FKP2_MKS2_MKP2, symbol Device:C
- added J1: ~, plc14500:PLC14500-Expansion, symbol plc14500:PLC14500-Expansion
- added unit 7 of U1
- added unit 3 of U3
- added unit 7 of U3
- added U?: 74HC14, Package_DIP:DIP-14_W7.62mm_LongPads, symbol plc14500:74HC14
- C4: footprint Capacitor_THT:CP_Radial_D8.0mm_P5.00mm -> Capacitor_THT:CP_Radial_D5.0mm_P2.50mm; symbol plc14500-rescue:CP-Device -> plc14500:CP-Device
- D1, D10, D11, D12, D13, D14, D15, D16, D2, D3, D4, D5, D6, D7, D8, D9: symbol plc14500-rescue:LED5MM-SparkFun-LED -> plc14500:LED; Field4 XXX-00000 -> (none)
- RV1: symbol plc14500-rescue:R_POT_TRIM-Device -> plc14500:Trimmer
- S12, S13, S14, S5, S6, S7, S8: symbol plc14500-rescue:SWITCH-DPDT-PTH-GPI-152-3013-SparkFun-Switches -> plc14500:SWITCH-DPDT
- U1, U3, U?: symbol 74xx:74HC14 -> plc14500:74HC14
- U2: symbol 4xxx:4051 -> plc14500:4051
- U?: symbol plc14500-rescue:555D-SparkFun-IC-Special-Function -> plc14500:555
Connections:
- net +5V: now also C3.1, C1.2, C2.2, J1.18 (+5v), U1.14 (VCC), U3.14 (VCC); no longer C3.2
- net GND: now also C3.2, S12.8 (GND), S12.9 (GND), S13.8 (GND), S13.9 (GND), S14.8 (GND), S14.9 (GND), S5.8 (GND), S5.9 (GND), S6.8 (GND), S6.9 (GND), S7.8 (GND), S7.9 (GND), S8.8 (GND), S8.9 (GND), C1.1, C2.1, J1.8 (GND), U1.7 (GND), U3.7 (GND); no longer C3.1
- net RES: now also J1.17 (RST)
- net TMR0-TRG: now also J1.16 (OUT7)
- net OUT1: now reaches D15.A, U5.10 (Q1)
- net OUT1: now also J1.10 (OUT1)
- net OUT2: now reaches D14.A, U5.11 (Q2)
- net OUT2: now also J1.11 (OUT2)
- net OUT3: now reaches D13.A, U5.12 (Q3)
- net OUT3: now also J1.12 (OUT3)
- net OUT4: now reaches D12.A, U5.13 (Q4)
- net OUT4: now also J1.13 (OUT4)
- net OUT5: now reaches D11.A, U5.14 (Q5)
- net OUT5: now also J1.14 (OUT5)
- net OUT6: now reaches D10.A, U5.15 (Q6)
- net OUT6: now also J1.15 (OUT6)
- net OUT0: now reaches D16.A, U5.9 (Q0)
- net OUT0: now also J1.9 (OUT0)
- net at S5.1: now also S5.5, S5.7, U1.1; no longer U1.2
- net at S5.3: now also U1.2; no longer S5.7
- net EXTIN0: now reaches R1.2, S1.1, S5.6
- net EXTIN0: now also J1.1 (EXTIN0)
- net at S6.1: now also S6.5, S6.7, U1.3; no longer U1.4
- net at S6.3: now also U1.4; no longer S6.7
- net EXTIN1: now reaches R2.2, S2.1, S6.6
- net EXTIN1: now also J1.2 (EXTIN1)
- net at S7.1: now also S7.5, S7.7, U1.5; no longer U1.6
- net at S7.3: now also U1.6; no longer S7.7
- net EXTIN2: now reaches R3.2, S3.1, S7.6
- net EXTIN2: now also J1.3 (EXTIN2)
- net at S8.1: now also S8.5, S8.7, U1.9; no longer U1.8
- net at S8.3: now also U1.8; no longer S8.7
- net EXTIN3: now reaches R4.2, S4.1, S8.6
- net EXTIN3: now also J1.4 (EXTIN3)
- net at S12.1: now also S12.5; no longer U1.10
- net at S12.3: now also U1.10; no longer S12.7
- net at U1.11: now also S12.7; no longer S12.5
- net EXTIN4: now reaches R9.2, S12.6, S9.1
- net EXTIN4: now also J1.5 (EXTIN4)
- net at S13.1: now also S13.5; no longer U1.12
- net at S13.3: now also U1.12; no longer S13.7
- net at U1.13: now also S13.7; no longer S13.5
- net EXTIN5: now reaches R10.2, S10.1, S13.6
- net EXTIN5: now also J1.6 (EXTIN5)
- net at S14.1: now also S14.5; no longer U3.2
- net at S14.3: now also U3.2; no longer S14.7
- net at U3.1: now also S14.7; no longer S14.5
- net EXTIN6: now reaches R11.2, S11.1, S14.6
- net EXTIN6: now also J1.7 (EXTIN6)
- net IN-WINH renamed IN-INH
- no-connect marks 10 -> 6
Other:
- note added: "Expansion"
- note added: "Input Selector"
- note added: "Output Latch"
- note removed: "Input"
- note removed: "Output"
- note removed: "Programming I/F"
- moved on the sheet: C3, C4, C5, C6, D1, D10, D11, D12, D13, D14, D15, D16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
