File: board/plc14500/SPRAM.kicad_sch (KiCad schematic)
At the start: 26 parts, among them U12 4011, U13 4099, U14 4051

Commit message: Feature/rev.d (#19)
* First tests for a rust upload tool, WIP

* Rearrange LEDs

* Remove kicad backups

* REV.D Schema updates

* Restore PCB anchoring holes

* Address ERC errors

* Cleanup, ready to route

* REV.D first proto

* Fix issues on REV.D0

* REV.D schema fixes, better assembler output, some docs

* Add ignore of kicad lock files

* Fixes

* route

* Re-route REV.D, fab files next round

* Re-route REV.D, fab files next round

* Rev.d

* Added reset cap from program line

* REV.D artifacts

* Cleanup REV.D

* Remove old file
Parts:
- removed C?: 100nF, Capacitor_THT:C_Rect_L7.2mm_W2.5mm_P5.00mm_FKS2_FKP2_MKS2_MKP2, symbol Device:C
- removed U? (x2): 74HC14, Package_DIP:DIP-14_W7.62mm_LongPads, symbol 74xx:74HC14
- added C? (x3): 100nF, Capacitor_THT:C_Rect_L7.2mm_W2.5mm_P5.00mm_FKS2_FKP2_MKS2_MKP2, symbol Device:C
- added U? (x3): 74HC14, Package_DIP:DIP-14_W7.62mm_LongPads, symbol plc14500:74HC14
- added U?: 4011, Package_DIP:DIP-14_W7.62mm_LongPads, symbol plc14500:4011
- D43, D44, D45, D46, D47, D48, D49: symbol plc14500-rescue:LED5MM-SparkFun-LED -> plc14500:LED; Field4 XXX-00000 -> (none)
- R59: value 3K3 -> 820R
- U12: symbol 4xxx:4011 -> plc14500:4011
- U14: symbol 4xxx:4051 -> plc14500:4051
- U? (x3): symbol 74xx:74HC14 -> plc14500:74HC14
Connections:
- net +5V: now also C?.2, C?.2, U?.14 (VCC)
- net GND: now also C?.1, C?.1, U?.7 (GND)
- net W: now also C?.2
- net at R59.2: now also C?.1, U?.3
- net at U12.2, U12.5: now also U?.4
- net IN-WINH renamed IN-INH
- net SPRAM-WINH renamed SPRAM-INH
- net SRAM-WD renamed SPRAM-WD
- new net: U?.3, U?.4
Other:
- note added: "*1) Prior to REV.C this was a generic SPR and connected to Q7 of U13. This means software running on boards prior to REV.C were unaable to instrospect on the value of RR."
- note added: "IN-INH"
- note added: "SPRAM-INH"
- note added: "SPRAM-WD"
- note added: "W - Is the Write line from the MC14500. When asserted the processor wants to write out D. The 4 lines from the Write Line Glue logic address what is being written to or read from. D7 is the msb of the program byte currently executed and addresses the I/O if set or the SPRAM is clear. IN-INH and SPRAM-INH control the INH line of the input sekector and SPRAM selector respectively. When asserted the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"
- note removed: "*1) Prior to REV.C this was a generic SPR and connected to Q7 of U13"
- note removed: "IN-WINH"
- note removed: "SRAM-WD"
- note removed: "SRAM-WINH"
- company: (none) -> Nicola Cimmino
- title: Scratchpad RAM -> PLC14500 - Nano
- moved on the sheet: C?, D43, D44, D45, D46, D47, D48, D49, R60, R61, R62, R63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
