File: board/plc14500/programming_if.kicad_sch (KiCad schematic)
At the start: 7 parts, among them U3 74HC14, U6 Arduino Nano

Commit message: Fix/rst line (#20)
* Clear OUT and SPR on program

* Fix RST line pulsing on program upload doesn't work

* Bump bootloader version to 1.3
Parts:
- removed C20: 1uF NP, Capacitor_THT:C_Radial_D6.3mm_H5.0mm_P2.50mm, symbol Device:C_Small
Other:
- note added: "NOTE! A6 is input only so the bootloader is unable to pulse RST. However RST is read by the bootloader to allow using the RST button to enter bootloader options mode."
Changed lines of the file:
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@@
     (comment 1 "REV.D")
-  )
-  (junction (at 148.59 103.505) (diameter 0) (color 0 0 0 0)
   )
   (junction (at 160.655 103.505) (diameter 0) (color 0 0 0 0)
@@
     (stroke (width 0) (type default))
   )
-  (wire (pts (xy 148.59 90.805) (xy 148.59 92.71))
-    (stroke (width 0) (type default))
-  )
-  (wire (pts (xy 139.065 103.505) (xy 148.59 103.505))
-    (stroke (width 0) (type default))
-  )
   (wire (pts (xy 160.655 84.455) (xy 161.925 84.455))
     (stroke (width 0) (type default))
@@
     (stroke (width 0) (type default))
   )
-  (wire (pts (xy 148.59 103.505) (xy 160.655 103.505))
+  (wire (pts (xy 139.065 103.505) (xy 160.655 103.505))
     (stroke (width 0) (type default))
   )
@@
     (stroke (width 0) (type default))
   )
-  (wire (pts (xy 146.685 90.805) (xy 148.59 90.805))
-    (stroke (width 0) (type default))
-  )
   (wire (pts (xy 83.82 90.805) (xy 78.74 90.805))
     (stroke (width 0) (type default))
@@
     (stroke (width 0) (type default))
   )
-  (wire (pts (xy 148.59 97.79) (xy 148.59 103.505))
-    (stroke (width 0) (type default))
-  )
   (wire (pts (xy 97.79 113.665) (xy 99.06 113.665))
     (stroke (width 0) (type default))
@@
   (wire (pts (xy 97.79 114.935) (xy 97.79 113.665))
     (stroke (width 0) (type default))
+  )
+  (text "NOTE! A6 is input only so the bootloader is unable to\npulse RST. However RST is read by the bootloader to allow\nusing the RST button to enter bootloader options mode."
+    (at 76.835 124.46 0)
+    (effects (font (size 1.27 1.27)) (justify left bottom))
   )
   (text "The programmer asserts the PRG line to take control of the bus. This causes the PC address lines to go to HiZ.\n\n!WEN is cleared by the programmer once each program byte value and address is stable. This triggers a write in RAM.\n\nThe programmer, or the user, can assert the RES line to cause a reset of the PC and of the lataches."
@@
   (hierarchical_label "A5" (shape output) (at 119.38 90.805 0) (fields_autoplaced)
     (effects (font (size 1.27 1.27)) (justify left))
-  )
-  (hierarchical_label "PRG" (shape output) (at 146.685 90.805 180) (fields_autoplaced)
-    (effects (font (size 1.27 1.27)) (justify right))
   )
   (hierarchical_label "!WEN" (shape output) (at 119.38 100.965 0) (fields_autoplaced)
@@
         )
       )
-    )
-  )
-  (symbol (lib_id "Device:C_Small") (at 148.59 95.25 0) (unit 1)
-    (in_bom yes) (on_board yes) (dnp no) (fields_autoplaced)
-    (property "Reference" "C20" (at 151.13 93.9863 0)
-      (effects (font (size 1.27 1.27)) (justify left))
-    )
-    (property "Value" "1uF NP" (at 151.13 96.5263 0)
-      (effects (font (size 1.27 1.27)) (justify left))
-    )
-    (property "Footprint" "Capacitor_THT:C_Radial_D6.3mm_H5.0mm_P2.50mm" (at 148.59 95.25 0)
-      (effects (font (size 1.27 1.27)) hide)
-    )
-    (property "Datasheet" "~" (at 148.59 95.25 0)
-      (effects (font (size 1.27 1.27)) hide)
-    )
-    (pin "1")
-    (pin "2")
-    (instances
-      (project "plc14500"
-        (path "/e5c24396-229a-4727-a88d-8f28d7f70179/8308f4d3-970f-416c-a310-08d544e11abe"
-          (reference "C20") (unit 1)
-        )
-      )
